File: PCB/M5_BuggyProject/M5_BuggyProject.kicad_pcb (KiCad board)
At the start: 2 copper layers, 0 parts

Commit message: Added updated netlist, started PCB
Parts:
- added A1: Feather 328P, Module:Adafruit_Feather, F.Cu at (125.7, 63.5)
- added A2: DRV8871, Connector_PinSocket_2.54mm:PinSocket_1x04_P2.54mm_Vertical, F.Cu at (153.6, 63.5)
- added A3: DRV8871, Connector_PinSocket_2.54mm:PinSocket_1x04_P2.54mm_Vertical, F.Cu at (153.7, 78.7)
- added A4: DRV8871, Connector_PinSocket_2.54mm:PinSocket_1x04_P2.54mm_Vertical, F.Cu at (153.7, 94.0)
- added A5: DRV8871, Connector_PinSocket_2.54mm:PinSocket_1x04_P2.54mm_Vertical, F.Cu at (118.1, 63.5)
- added A6: DRV8871, Connector_PinSocket_2.54mm:PinSocket_1x04_P2.54mm_Vertical, F.Cu at (118.1, 78.7)
- added A7: DRV8871, Connector_PinSocket_2.54mm:PinSocket_1x04_P2.54mm_Vertical, F.Cu at (118.1, 94.0)
- added D1: D_Schottky, Package_TO_SOT_THT:TO-220-2_Horizontal_TabDown, F.Cu at (116.8, 114.3)
- added J1: XT60, Connector_AMASS:AMASS_XT60-F_1x02_P7.20mm_Vertical, F.Cu at (153.7, 111.8)
Routing:
- net AIN2: track 0.00 -> 0.80 mm
