File: PCB/M5_BuggyProject/M5_BuggyProject.sch (KiCad schematic (older format))
At the start: 15 parts, among them J1 XT60

Commit message: Changed firmware, updated schematic and README
Parts:
- removed D3: SIG, symbol Device:LED
- removed D4: NO_SIG, symbol Device:LED
- removed R1, R2: 330, symbol Device:R
Connections:
- wire segments 55 -> 52
- no-connect marks 19 -> 21
Other:
- moved on the sheet: A1
Changed lines of the file:
@@
 Text Notes 1000 950  0    75   ~ 0
 Power Electronics\n
-NoConn ~ 2950 3700
-NoConn ~ 2950 4200
-NoConn ~ 2950 4100
-NoConn ~ 2950 4000
-NoConn ~ 1950 4200
-NoConn ~ 1950 4100
-NoConn ~ 1950 4000
-NoConn ~ 1950 3800
-NoConn ~ 1950 3700
+NoConn ~ 2400 3750
+NoConn ~ 2400 4250
+NoConn ~ 2400 4150
+NoConn ~ 2400 4050
+NoConn ~ 1400 4250
+NoConn ~ 1400 4150
+NoConn ~ 1400 4050
+NoConn ~ 1400 3850
+NoConn ~ 1400 3750
 $Comp
 L Buggy_Components:VM #PWR010
@@
 	1    0    0    -1
 $EndComp
-Wire Wire Line
-	1150 3500 1950 3500
-Wire Wire Line
-	1500 3600 1950 3600
-Wire Wire Line
-	1150 3600 1150 3500
 Text Notes 5500 1450 0    75   ~ 0
 Control Electronics
@@
 	7500 4000 7500 1500
 Wire Notes Line
-	3500 2500 3500 5500
-Wire Notes Line
 	1000 5500 1000 2500
-Wire Notes Line
-	3500 5500 1000 5500
-Wire Notes Line
-	3500 2500 1000 2500
-$Comp
-L power:GND #PWR0103
-U 1 1 61D9CEC9
-P 1500 4200
-F 0 "#PWR0103" H 1500 3950 50  0001 C CNN
-F 1 "GND" H 1505 4027 50  0000 C CNN
-F 2 "" H 1500 4200 50  0001 C CNN
-F 3 "" H 1500 4200 50  0001 C CNN
-	1    1500 4200
-	1    0    0    -1
-$EndComp
-$Comp
-L power:GND #PWR0102
-U 1 1 61D9C867
-P 1150 4200
-F 0 "#PWR0102" H 1150 3950 50  0001 C CNN
-F 1 "GND" H 1155 4027 50  0000 C CNN
-F 2 "" H 1150 4200 50  0001 C CNN
-F 3 "" H 1150 4200 50  0001 C CNN
-	1    1150 4200
-	1    0    0    -1
-$EndComp
-$Comp
-L Device:R R1
-U 1 1 61D9A79A
-P 1150 3750
-F 0 "R1" H 1220 3796 50  0000 L CNN
-F 1 "330" H 1220 3705 50  0000 L CNN
-F 2 "" V 1080 3750 50  0001 C CNN
-F 3 "~" H 1150 3750 50  0001 C CNN
-	1    1150 3750
-	1    0    0    -1
-$EndComp
-$Comp
-L Device:R R2
-U 1 1 61D99D67
-P 1500 3750
-F 0 "R2" H 1570 3796 50  0000 L CNN
-F 1 "330" H 1570 3705 50  0000 L CNN
-F 2 "" V 1430 3750 50  0001 C CNN
-F 3 "~" H 1500 3750 50  0001 C CNN
-	1    1500 3750
-	1    0    0    -1
-$EndComp
-$Comp
-L Device:LED D4
-U 1 1 61D8850F
-P 1500 4050
-F 0 "D4" V 1539 3932 50  0000 R CNN
-F 1 "NO_SIG" V 1448 3932 50  0000 R CNN
-F 2 "" H 1500 4050 50  0001 C CNN
-F 3 "~" H 1500 4050 50  0001 C CNN
-	1    1500 4050
-	0    -1   -1   0
-$EndComp
-$Comp
-L Device:LED D3
-U 1 1 61D86F74
-P 1150 4050
-F 0 "D3" V 1189 3932 50  0000 R CNN
-F 1 "SIG" V 1098 3932 50  0000 R CNN
-F 2 "" H 1150 4050 50  0001 C CNN
-F 3 "~" H 1150 4050 50  0001 C CNN
-	1    1150 4050
-	0    -1   -1   0
-$EndComp
-NoConn ~ 1950 4800
-NoConn ~ 1950 4700
-NoConn ~ 1950 4500
-NoConn ~ 1950 4400
-NoConn ~ 2950 3500
-NoConn ~ 2950 3400
-NoConn ~ 2950 3100
-NoConn ~ 2650 2700
-NoConn ~ 2550 2700
-NoConn ~ 2350 2700
+NoConn ~ 1400 4850
+NoConn ~ 1400 4750
+NoConn ~ 1400 4550
+NoConn ~ 1400 4450
+NoConn ~ 2400 3550
+NoConn ~ 2400 3450
+NoConn ~ 2400 3150
+NoConn ~ 2100 2750
+NoConn ~ 2000 2750
+NoConn ~ 1800 2750
 $Comp
 L power:GND #PWR0101
 U 1 1 61D8BB98
-P 2450 5200
-F 0 "#PWR0101" H 2450 4950 50  0001 C CNN
-F 1 "GND" H 2455 5027 50  0000 C CNN
-F 2 "" H 2450 5200 50  0001 C CNN
-F 3 "" H 2450 5200 50  0001 C CNN
-	1    2450 5200
+P 1900 5250
+F 0 "#PWR0101" H 1900 5000 50  0001 C CNN
+F 1 "GND" H 1905 5077 50  0000 C CNN
+F 2 "" H 1900 5250 50  0001 C CNN
+F 3 "" H 1900 5250 50  0001 C CNN
+	1    1900 5250
 	1    0    0    -1
 $EndComp
@@
 L MCU_Module:Adafruit_Feather_328P A1
 U 1 1 61D69E86
-P 2450 3900
-F 0 "A1" H 2100 5050 50  0000 C CNN
-F 1 "Feather 328P" H 2700 2650 40  0000 C CNN
-F 2 "Module:Adafruit_Feather" H 2550 2550 50  0001 L CNN
-F 3 "https://cdn-learn.adafruit.com/downloads/pdf/adafruit-feather.pdf" H 2450 3100 50  0001 C CNN
-	1    2450 3900
-	1    0    0    -1
-$EndComp
-Text GLabel 2950 3900 2    50   Input ~ 0
+P 1900 3950
+F 0 "A1" H 1550 5100 50  0000 C CNN
+F 1 "Feather 328P" H 2150 2700 40  0000 C CNN
+F 2 "Module:Adafruit_Feather" H 2000 2600 50  0001 L CNN
+F 3 "https://cdn-learn.adafruit.com/downloads/pdf/adafruit-feather.pdf" H 1900 3150 50  0001 C CNN
+	1    1900 3950
+	1    0    0    -1
+$EndComp
+Text GLabel 2400 3950 2    50   Input ~ 0
 CHANNEL_2
-Text GLabel 2950 3800 2    50   Input ~ 0
+Text GLabel 2400 3850 2    50   Input ~ 0
 CHANNEL_1
-Text GLabel 1950 3400 0    50   Input ~ 0
+Text GLabel 1400 3450 0    50   Input ~ 0
 BIN2
-Text GLabel 1950 3300 0    50   Input ~ 0
+Text GLabel 1400 3350 0    50   Input ~ 0
 BIN1
-Text GLabel 1950 3200 0    50   Input ~ 0
+Text GLabel 1400 3250 0    50   Input ~ 0
 AIN2
-Text GLabel 1950 3100 0    50   Input ~ 0
+Text GLabel 1400 3150 0    50   Input ~ 0
 AIN1
 Connection ~ 6800 3550
@@
 Wire Notes Line
 	1000 2000 3500 2000
+NoConn ~ 1400 3550
+NoConn ~ 1400 3650
+Wire Notes Line
+	3000 2500 3000 5500
+Wire Notes Line
+	1000 2500 3000 2500
+Wire Notes Line
+	1000 5500 3000 5500
 $EndSCHEMATC

Commit message: Added updated netlist, started PCB
Parts:
- removed C1: 2200uF, symbol Device:CP
- removed D2: D_Zener, symbol Device:D_Zener
- D1: footprint (none) -> Package_TO_SOT_THT:TO-220-2_Horizontal_TabDown
- J1: footprint (none) -> Connector_AMASS:AMASS_XT60-F_1x02_P7.20mm_Vertical
Connections:
- net labels added: +7.5V
- net labels removed: VM
- wire segments 52 -> 51
Other:
- moved on the sheet: A1, A2, A3, A4, A5, A6, A7

Commit message: Added labels, traces for controls
Other:
- moved on the sheet: D1
Changed lines of the file:
@@
-$EndComp
-$Comp
-L power:VCC #PWR04
-U 1 1 61DEDB89
-P 2000 1400
-F 0 "#PWR04" H 2000 1250 50  0001 C CNN
-F 1 "VCC" H 2015 1573 50  0000 C CNN
-F 2 "" H 2000 1400 50  0001 C CNN
-F 3 "" H 2000 1400 50  0001 C CNN
-	1    2000 1400
-	1    0    0    -1
 $EndComp
 $Comp
 L Device:D_Schottky D1
 U 1 1 61DEEBD5
-P 2300 1400
-F 0 "D1" H 2300 1183 50  0000 C CNN
-F 1 "D_Schottky" H 2300 1274 40  0000 C CNN
-F 2 "Package_TO_SOT_THT:TO-220-2_Horizontal_TabDown" H 2300 1400 50  0001 C CNN
-F 3 "~" H 2300 1400 50  0001 C CNN
-	1    2300 1400
+P 2000 1400
+F 0 "D1" H 2000 1183 50  0000 C CNN
+F 1 "D_Schottky" H 2000 1274 40  0000 C CNN
+F 2 "Package_TO_SOT_THT:TO-220-2_Horizontal_TabDown" H 2000 1400 50  0001 C CNN
+F 3 "~" H 2000 1400 50  0001 C CNN
+	1    2000 1400
 	-1   0    0    1
 $EndComp
@@
 Text GLabel 1400 3300 0    50   Input ~ 0
 BIN1
-Text GLabel 1400 3200 0    50   Input ~ 0
-AIN2
-Text GLabel 1400 3100 0    50   Input ~ 0
-AIN1
 Connection ~ 7300 3050
 Wire Wire Line
@@
 Wire Notes Line
 	1000 2500 3000 2500
-Wire Wire Line
-	2150 1400 2000 1400
 $Comp
 L power:+7.5V #PWR06
 U 1 1 61DEFD0D
-P 2600 1400
-F 0 "#PWR06" H 2600 1250 50  0001 C CNN
-F 1 "+7.5V" H 2615 1573 50  0000 C CNN
-F 2 "" H 2600 1400 50  0001 C CNN
-F 3 "" H 2600 1400 50  0001 C CNN
-	1    2600 1400
-	1    0    0    -1
-$EndComp
-Wire Wire Line
-	2450 1400 2600 1400
+P 2300 1400
+F 0 "#PWR06" H 2300 1250 50  0001 C CNN
+F 1 "+7.5V" H 2315 1573 50  0000 C CNN
+F 2 "" H 2300 1400 50  0001 C CNN
+F 3 "" H 2300 1400 50  0001 C CNN
+	1    2300 1400
+	1    0    0    -1
+$EndComp
+Wire Wire Line
+	2150 1400 2300 1400
 $Comp
 L power:+7.5V #PWR07
@@
 	1    0    0    -1
 $EndComp
+Wire Wire Line
+	1850 1400 1700 1400
+$Comp
+L power:VCC #PWR0102
+U 1 1 61DE024E
+P 1700 1400
+F 0 "#PWR0102" H 1700 1250 50  0001 C CNN
+F 1 "VCC" H 1715 1573 50  0000 C CNN
+F 2 "" H 1700 1400 50  0001 C CNN
+F 3 "" H 1700 1400 50  0001 C CNN
+	1    1700 1400
+	1    0    0    -1
+$EndComp
+Text GLabel 1400 3100 0    50   Input ~ 0
+AIN2
+Text GLabel 1400 3200 0    50   Input ~ 0
+AIN1
 $EndSCHEMATC

Commit message: Updated PCB, added Digikey footprint library
Parts:
- added C1: 2200uF, Capacitor_THT:CP_Radial_D10.0mm_P5.00mm, symbol Device:CP
- added D3: LED, LED_SMD:LED_1206_3216Metric, symbol Device:LED
- added R1: 698, Resistor_SMD:R_1206_3216Metric, symbol Device:R
- added Z1: Diode, digikey-footprints:DO-214AC, symbol dk_Diodes-Zener-Single:1N5231BTR
- D1: footprint Package_TO_SOT_THT:TO-220-2_Horizontal_TabDown -> Package_TO_SOT_THT:TO-220-2_Vertical
- J1: footprint Connector_AMASS:AMASS_XT60-F_1x02_P7.20mm_Vertical -> Connector_AMASS:AMASS_XT60-M_1x02_P7.20mm_Vertical
Connections:
- net labels added: +12V
- net labels removed: +7.5V
- wire segments 51 -> 52
Other:
- moved on the sheet: A2, A3, A4, A5, A6, A7, D1, J1

Commit message: Finalised PCB for v1.0
Parts:
- added BZ1: BEEP, Buzzer_Beeper:Buzzer_12x9.5RM7.6, symbol Device:Buzzer
- added D2, D4: ORANGE, LED_SMD:LED_1206_3216Metric, symbol Device:LED
- added H1, H2, H3, H4: M, MountingHole:MountingHole_3.2mm_M3_Pad_Via, symbol Mechanical:MountingHole_Pad
- added J2: VCC, TestPoint:TestPoint_Loop_D1.80mm_Drill1.0mm_Beaded, symbol Connector:Conn_01x01_Male
- added J3: 10V, TestPoint:TestPoint_Loop_D1.80mm_Drill1.0mm_Beaded, symbol Connector:Conn_01x01_Male
- added R2, R3: 100, Resistor_SMD:R_1206_3216Metric, symbol Device:R
- D3: value LED -> BLUE
- R1: value 698 -> 330
Connections:
- net labels added: +10V, BEEP, CHANNEL_3, CONFIG_L, CONFIG_R
- net labels removed: +12V
- wire segments 52 -> 55
- no-connect marks 21 -> 17
Other:
- note added: "Control Electronics / Drivetrain"
- note added: "Debugging"
- note added: "Mounting Holes"
- note removed: "Control Electronics"
- moved on the sheet: A1, A2, A3, A4, A5, A6, A7, C1, D1, D3, R1

Commit message: Added connector for radio receiver
Parts:
- added J4: RF Receiver, Connector_PinSocket_2.54mm:PinSocket_1x05_P2.54mm_Vertical, symbol Connector:Conn_01x05_Female
- Z1: symbol dk_Diodes-Zener-Single:1N5231BTR -> M5_BuggyProject-rescue:1N5231BTR-dk_Diodes-Zener-Single
Connections:
- net labels added: +3.3V, +5V
- wire segments 55 -> 59
- no-connect marks 17 -> 15
Other:
- note added: "MCU Connections"
- note removed: "Debugging"
- moved on the sheet: A1
Changed lines of the file:
@@
 	1950 1300 2100 1300
 $Comp
-L dk_Diodes-Zener-Single:1N5231BTR Z1
+L M5_BuggyProject-rescue:1N5231BTR-dk_Diodes-Zener-Single Z1
 U 1 1 61DF337E
 P 2500 1500
@@
 	1    0    0    -1
 $EndComp
+Text GLabel 1450 3250 0    50   Input ~ 0
+AIN1
 Text GLabel 1450 3150 0    50   Input ~ 0
-AIN1
-Text GLabel 1450 3050 0    50   Input ~ 0
 AIN2
-NoConn ~ 1450 4050
+NoConn ~ 1450 4150
 Wire Notes Line
 	1000 5500 3000 5500
+Text GLabel 2450 3950 2    50   Input ~ 0
+CHANNEL_2
 Text GLabel 2450 3850 2    50   Input ~ 0
-CHANNEL_2
-Text GLabel 2450 3750 2    50   Input ~ 0
 CHANNEL_1
 $Comp
 L MCU_Module:Adafruit_Feather_328P A1
 U 1 1 61D69E86
-P 1950 3850
-F 0 "A1" H 1600 5000 50  0000 C CNN
-F 1 "Feather 328P" H 2200 2600 40  0000 C CNN
-F 2 "Module:Adafruit_Feather" H 2050 2500 50  0001 L CNN
-F 3 "https://cdn-learn.adafruit.com/downloads/pdf/adafruit-feather.pdf" H 1950 3050 50  0001 C CNN
-	1    1950 3850
-	1    0    0    -1
-$EndComp
-NoConn ~ 1450 3450
-Text GLabel 1450 3250 0    50   Input ~ 0
+P 1950 3950
+F 0 "A1" H 1600 5100 50  0000 C CNN
+F 1 "Feather 328P" H 2200 2700 40  0000 C CNN
+F 2 "Module:Adafruit_Feather" H 2050 2600 50  0001 L CNN
+F 3 "https://cdn-learn.adafruit.com/downloads/pdf/adafruit-feather.pdf" H 1950 3150 50  0001 C CNN
+	1    1950 3950
+	1    0    0    -1
+$EndComp
+NoConn ~ 1450 3550
+Text GLabel 1450 3350 0    50   Input ~ 0
 BIN1
-Text GLabel 1450 3350 0    50   Input ~ 0
+Text GLabel 1450 3450 0    50   Input ~ 0
 BIN2
 $Comp
 L power:GND #PWR0101
 U 1 1 61D8BB98
-P 1950 5150
-F 0 "#PWR0101" H 1950 4900 50  0001 C CNN
-F 1 "GND" H 1955 4977 50  0000 C CNN
-F 2 "" H 1950 5150 50  0001 C CNN
-F 3 "" H 1950 5150 50  0001 C CNN
-	1    1950 5150
-	1    0    0    -1
-$EndComp
-NoConn ~ 1850 2650
-NoConn ~ 2050 2650
-NoConn ~ 2150 2650
-NoConn ~ 2450 3050
-NoConn ~ 2450 3350
+P 1950 5250
+F 0 "#PWR0101" H 1950 5000 50  0001 C CNN
+F 1 "GND" H 1955 5077 50  0000 C CNN
+F 2 "" H 1950 5250 50  0001 C CNN
+F 3 "" H 1950 5250 50  0001 C CNN
+	1    1950 5250
+	1    0    0    -1
+$EndComp
+NoConn ~ 1850 2750
+NoConn ~ 2450 3150
 NoConn ~ 2450 3450
-NoConn ~ 1450 4350
+NoConn ~ 2450 3550
 NoConn ~ 1450 4450
-NoConn ~ 1450 4650
+NoConn ~ 1450 4550
 NoConn ~ 1450 4750
-NoConn ~ 1450 3650
+NoConn ~ 1450 4850
 NoConn ~ 1450 3750
-NoConn ~ 1450 3950
-NoConn ~ 1450 4150
-NoConn ~ 2450 3650
+NoConn ~ 1450 3850
+NoConn ~ 1450 4050
+NoConn ~ 1450 4250
+NoConn ~ 2450 3750
 Wire Notes Line
 	5500 2000 4500 2000
@@
 	1    0    0    -1
 $EndComp
-Text GLabel 2450 4050 2    50   Input ~ 0
+Text GLabel 2450 4150 2    50   Input ~ 0
 CONFIG_L
-Text GLabel 2450 4150 2    50   Input ~ 0
+Text GLabel 2450 4250 2    50   Input ~ 0
 CONFIG_R
-Text GLabel 1450 3550 0    50   Input ~ 0
+Text GLabel 1450 3650 0    50   Input ~ 0
 BEEP
-Wire Notes Line
-	3500 4000 3500 2500
 $Comp
 L Device:LED D4
@@
 $EndComp
 Wire Notes Line
-	5500 2500 5500 4000
-Wire Notes Line
 	3500 2500 5500 2500
-Wire Notes Line
-	3500 4000 5500 4000
 $Comp
 L Device:R R2
@@
 Connection ~ 7300 3050
 Text Notes 3500 2450 0    75   ~ 0
-Debugging
-Text GLabel 2450 3950 2    50   Input ~ 0
+MCU Connections
+Text GLabel 2450 4050 2    50   Input ~ 0
 CHANNEL_3
 $Comp
@@
 	1    0    0    -1
 $EndComp
+$Comp
+L Connector:Conn_01x05_Female J4
+U 1 1 61F7AADA
+P 4500 4300
+F 0 "J4" V 4346 4548 50  0000 L CNN
+F 1 "RF Receiver" V 4437 4548 50  0000 L CNN
+F 2 "Connector_PinSocket_2.54mm:PinSocket_1x05_P2.54mm_Vertical" H 4500 4300 50  0001 C CNN
+F 3 "~" H 4500 4300 50  0001 C CNN
+	1    4500 4300
+	0    1    1    0
+$EndComp
+Wire Wire Line
+	4500 4100 4500 3900
+Wire Wire Line
+	4500 3900 4300 3900
+Wire Wire Line
+	4400 4100 4400 4000
+Wire Wire Line
+	4400 4000 4300 4000
+Text GLabel 4300 3900 0    50   Input ~ 0
+CHANNEL_3
+Text GLabel 4300 4000 0    50   Input ~ 0
+CHANNEL_2
+Text GLabel 4300 4100 0    50   Input ~ 0
+CHANNEL_1
+$Comp
+L power:GND #PWR023
+U 1 1 61F82930
+P 4700 4100
+F 0 "#PWR023" H 4700 3850 50  0001 C CNN
+F 1 "GND" H 4705 3927 50  0000 C CNN
+F 2 "" H 4700 4100 50  0001 C CNN
+F 3 "" H 4700 4100 50  0001 C CNN
+	1    4700 4100
+	-1   0    0    1
+$EndComp
+$Comp
+L power:+3.3V #PWR020
+U 1 1 61F83393
+P 2050 2750
+F 0 "#PWR020" H 2050 2600 50  0001 C CNN
+F 1 "+3.3V" H 2065 2923 50  0000 C CNN
+F 2 "" H 2050 2750 50  0001 C CNN
+F 3 "" H 2050 2750 50  0001 C CNN
+	1    2050 2750
+	1    0    0    -1
+$EndComp
+$Comp
+L power:+5V #PWR021
+U 1 1 61F86A6B
+P 2150 2750
+F 0 "#PWR021" H 2150 2600 50  0001 C CNN
+F 1 "+5V" V 2165 2878 50  0000 L CNN
+F 2 "" H 2150 2750 50  0001 C CNN
+F 3 "" H 2150 2750 50  0001 C CNN
+	1    2150 2750
+	0    1    1    0
+$EndComp
+$Comp
+L power:+5V #PWR022
+U 1 1 61F874D6
+P 4600 4100
+F 0 "#PWR022" H 4600 3950 50  0001 C CNN
+F 1 "+5V" V 4700 4100 50  0000 L CNN
+F 2 "" H 4600 4100 50  0001 C CNN
+F 3 "" H 4600 4100 50  0001 C CNN
+	1    4600 4100
+	0    -1   -1   0
+$EndComp
+Wire Notes Line
+	5500 4500 3500 4500
+Wire Notes Line
+	3500 2500 3500 4500
+Wire Notes Line
+	5500 2500 5500 4500
 $EndSCHEMATC

Commit message: Increased board size for trace width.
Parts:
- removed J4: RF Receiver, Connector_PinSocket_2.54mm:PinSocket_1x05_P2.54mm_Vertical, symbol Connector:Conn_01x05_Female
- added H5: MountingHole, symbol Mechanical:MountingHole
- added J4: Receiver, Connector_PinSocket_2.54mm:PinSocket_1x05_P2.54mm_Vertical, symbol Connector_Generic:Conn_01x05
- A1: symbol MCU_Module:Adafruit_Feather_328P -> M5_BuggyProject-rescue:Adafruit_Feather_328P-MCU_Module
Connections:
- net +3V3: now also J4.2 (Pin_2)
- net CHANNEL_1: now also J4.5 (Pin_5)
- net CHANNEL_2: now also J4.4 (Pin_4)
- net CHANNEL_3: now also J4.3 (Pin_3)
- net GND: now also J4.1 (Pin_1)
Changed lines of the file:
@@
 CHANNEL_1
 $Comp
-L MCU_Module:Adafruit_Feather_328P A1
+L M5_BuggyProject-rescue:Adafruit_Feather_328P-MCU_Module A1
 U 1 1 61D69E86
 P 1950 3950
@@
 $EndComp
 $Comp
-L Connector:Conn_01x05_Female J4
-U 1 1 61F7AADA
-P 4500 4300
-F 0 "J4" V 4346 4548 50  0000 L CNN
-F 1 "RF Receiver" V 4437 4548 50  0000 L CNN
-F 2 "Connector_PinSocket_2.54mm:PinSocket_1x05_P2.54mm_Vertical" H 4500 4300 50  0001 C CNN
-F 3 "~" H 4500 4300 50  0001 C CNN
-	1    4500 4300
-	0    1    1    0
-$EndComp
-Wire Wire Line
-	4500 4100 4500 3900
-Wire Wire Line
-	4500 3900 4300 3900
-Wire Wire Line
-	4400 4100 4400 4000
-Wire Wire Line
-	4400 4000 4300 4000
-Text GLabel 4300 3900 0    50   Input ~ 0
-CHANNEL_3
-Text GLabel 4300 4000 0    50   Input ~ 0
-CHANNEL_2
-Text GLabel 4300 4100 0    50   Input ~ 0
-CHANNEL_1
-$Comp
-L power:GND #PWR023
-U 1 1 61F82930
-P 4700 4100
-F 0 "#PWR023" H 4700 3850 50  0001 C CNN
-F 1 "GND" H 4705 3927 50  0000 C CNN
-F 2 "" H 4700 4100 50  0001 C CNN
-F 3 "" H 4700 4100 50  0001 C CNN
-	1    4700 4100
-	-1   0    0    1
-$EndComp
-$Comp
 L power:+3.3V #PWR020
 U 1 1 61F83393
@@
 	0    1    1    0
 $EndComp
-$Comp
-L power:+5V #PWR022
-U 1 1 61F874D6
-P 4600 4100
-F 0 "#PWR022" H 4600 3950 50  0001 C CNN
-F 1 "+5V" V 4700 4100 50  0000 L CNN
-F 2 "" H 4600 4100 50  0001 C CNN
-F 3 "" H 4600 4100 50  0001 C CNN
-	1    4600 4100
+Wire Notes Line
+	5500 4500 3500 4500
+Wire Notes Line
+	3500 2500 3500 4500
+Wire Notes Line
+	5500 2500 5500 4500
+$Comp
+L Connector_Generic:Conn_01x05 J4
+U 1 1 6201B3C5
+P 4500 4200
+F 0 "J4" V 4372 4480 50  0000 L CNN
+F 1 "Receiver" V 4463 4480 50  0000 L CNN
+F 2 "Connector_PinSocket_2.54mm:PinSocket_1x05_P2.54mm_Vertical" H 4500 4200 50  0001 C CNN
+F 3 "~" H 4500 4200 50  0001 C CNN
+	1    4500 4200
+	0    1    1    0
+$EndComp
+Text GLabel 4300 4000 0    50   Input ~ 0
+CHANNEL_1
+Wire Wire Line
+	4400 4000 4400 3900
+Wire Wire Line
+	4400 3900 4300 3900
+Text GLabel 4300 3900 0    50   Input ~ 0
+CHANNEL_2
+Wire Wire Line
+	4500 4000 4500 3800
+Wire Wire Line
+	4500 3800 4300 3800
+Text GLabel 4300 3800 0    50   Input ~ 0
+CHANNEL_3
+$Comp
+L power:+3.3V #PWR022
+U 1 1 62022951
+P 4600 4000
+F 0 "#PWR022" H 4600 3850 50  0001 C CNN
+F 1 "+3.3V" H 4615 4173 50  0000 C CNN
+F 2 "" H 4600 4000 50  0001 C CNN
+F 3 "" H 4600 4000 50  0001 C CNN
+	1    4600 4000
+	1    0    0    -1
+$EndComp
+$Comp
+L power:GND #PWR023
+U 1 1 62022B50
+P 4700 4000
+F 0 "#PWR023" H 4700 3750 50  0001 C CNN
+F 1 "GND" V 4705 3872 50  0000 R CNN
+F 2 "" H 4700 4000 50  0001 C CNN
+F 3 "" H 4700 4000 50  0001 C CNN
+	1    4700 4000
 	0    -1   -1   0
 $EndComp
-Wire Notes Line
-	5500 4500 3500 4500
-Wire Notes Line
-	3500 2500 3500 4500
-Wire Notes Line
-	5500 2500 5500 4500
+$Comp
+L Mechanical:MountingHole H5
+U 1 1 620461DC
+P 6700 4250
+F 0 "H5" H 6800 4296 50  0000 L CNN
+F 1 "MountingHole" H 6800 4205 50  0000 L CNN
+F 2 "" H 6700 4250 50  0001 C CNN
+F 3 "~" H 6700 4250 50  0001 C CNN
+	1    6700 4250
+	1    0    0    -1
+$EndComp
 $EndSCHEMATC
